File: 100mm-double-opposite-side/antmicro-alvium-flex-csi-adapter-100mm-double-opposite-side.sch (KiCad schematic (older format))
At the start: 3 parts, among them J1 WE_687622100002_FLEX, J2 WE_687622100002_FLEX, J3 WE_687650100002_FLEX

Commit message: 100mm-double-opposite: Add signage
Parts:
- added N1: oshw_logo, antmicro-footprints:oshw-logo, symbol antmicroMechanicalParts:oshw_logo
Other:
- note added: "Alvium Cameras"
- note added: "Alvium flex CSI adapter 100mm double opposite side contacts"
- note added: "Antmicro CSI interface"
- moved on the sheet: J1, J2, J3

Commit message: 100mm-double-opposite: update OSHW logotype
Parts:
- N1: footprint antmicro-footprints:oshw-logo -> antmicro-alvium-flex-csi-adapter-footprints:oshw-logo; symbol antmicroMechanicalParts:oshw_logo -> antmicro-alvium-flex-csi-adapter:oshw_logo
Changed lines of the file:
@@
 Alvium flex CSI adapter 100mm double opposite side contacts
 $Comp
-L antmicroMechanicalParts:oshw_logo N1
+L antmicro-alvium-flex-csi-adapter:oshw_logo N1
 U 1 1 5F89FCA6
 P 750 7500
 F 0 "N1" H 944 7503 50  0000 L CNN
 F 1 "oshw_logo" H 944 7412 50  0000 L CNN
-F 2 "antmicro-footprints:oshw-logo" H 770 7260 50  0001 C CNN
+F 2 "antmicro-alvium-flex-csi-adapter-footprints:oshw-logo" H 770 7260 50  0001 C CNN
 F 3 "" H 750 7500 50  0001 C CNN
 	1    750  7500
