File: 100mm-single-opposite-side/antmicro-alvium-flex-csi-adapter-100mm-single-opposite-side.sch (KiCad schematic (older format))
At the start: 2 parts, among them J1 WE_687622100002_FLEX, J2 WE_687650100002_FLEX

Commit message: 100mm-single-opposite: update signage
Parts:
- added N1: oshw_logo, antmicro-alvium-flex-csi-adapter-footprints:oshw-logo, symbol antmicro-alvium-flex-csi-adapter:oshw_logo
Other:
- note added: "Alvium Camera"
- note added: "Alvium flex CSI adapter 100mm single opposite side contacts"
- note added: "Antmicro CSI interface"
- note removed: "Antmicro - Alvium Flex CSI Adapter"
- note removed: "FFC contacts - Alvium side"
- note removed: "FFC contacts - Antmicro side"
- moved on the sheet: J1, J2
